File: Solar Panels/Solar Panels.kicad_pcb (KiCad board)
At the start: 2 copper layers, 113 x 82.5 mm, 58 parts, among them J2 5040500891

Commit message: Improve footprints, layout, routing
Parts:
- added J1: Conn_01x08_MountingPin, Connector_Molex:Molex_PicoBlade_53261-0871_1x08-1MP_P1.25mm_Horizontal, B.Cu at (183.0, 114.8)
- added J3: Conn_01x08_MountingPin, Connector_Molex:Molex_PicoBlade_53261-0871_1x08-1MP_P1.25mm_Horizontal, F.Cu at (85.9, 105.6)
- added J4: Conn_01x02, Connector_PinHeader_2.54mm:PinHeader_2x01_P2.54mm_Vertical, F.Cu at (85.4, 139.7)
- added J5: Conn_01x08_MountingPin, Connector_Molex:Molex_Pico-Lock_504050-0891_1x08-1MP_P1.50mm_Horizontal, B.Cu at (175.9, 115.0)
- J2: value 5040500891 -> Conn_01x08_MountingPin; footprint Solar Panel Library:5040500891 -> Connector_Molex:Molex_PicoBlade_53261-0871_1x08-1MP_P1.25mm_Horizontal
- moved J2 100.0 mm to (86.4, 125.1)
- moved JP5 4.24 mm to (151.6, 103.5)
- moved D7 2.01 mm to (176.5, 132.5)
- moved SC22 0.54 mm to (151.6, 135.8)
- moved SC23 0.46 mm to (132.5, 136.1)
- moved SC20 0.42 mm to (132.3, 128.0)
- moved SC16 0.42 mm to (162.0, 119.7)
- moved SC13 0.38 mm to (162.0, 111.6)
- moved SC19 0.33 mm to (162.0, 127.7)
- moved SC10 0.33 mm to (162.0, 103.5)
- moved SC7 0.30 mm to (151.2, 95.5)
- moved SC17 0.28 mm to (132.2, 120.0)
- moved SC25 0.27 mm to (151.5, 143.8)
- moved SC4 0.20 mm to (151.4, 87.4)
- moved SC26 0.20 mm to (132.3, 144.1)
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Routing:
- net +VDC: track 8.05 -> 36.2 mm, vias 2 -> 8
- net GND: track 16.4 -> 29.5 mm, vias 8 -> 13
- net Net-(SC26--): track 34.7 -> 44.7 mm, vias 0 -> 4
- net Net-(SC29--): track 35.1 -> 44.7 mm, vias 0 -> 4
- net Net-(SC5--): track 36.2 -> 44.7 mm, vias 0 -> 4
- net Net-(SC8--): track 36.3 -> 44.7 mm, vias 0 -> 4
- net Net-(SC20--): track 36.7 -> 44.9 mm, vias 0 -> 4
- net Net-(SC17--): track 36.8 -> 44.8 mm, vias 0 -> 4
- net Net-(SC2--): track 38.9 -> 44.9 mm, vias 0 -> 4
- net Net-(SC11--): track 39.0 -> 44.8 mm, vias 0 -> 4
- net Net-(SC14--): track 39.2 -> 44.7 mm, vias 0 -> 4
- net Net-(SC23--): track 39.2 -> 44.7 mm, vias 0 -> 4
- net Net-(SC19-+): track 10.0 -> 12.5 mm
- net Net-(JP5-A): track 4.09 -> 5.22 mm
- net Net-(JP7-A): track 4.62 -> 5.47 mm
Other:
- board text added: "Pre-Order Checks: * Hide reference designators. * Check that current can flow across the board in the top layer pour."
- board text added: "Spare DNP"
- board text added: "Stackup: 2 layers. 1.6mm FR4 PCB. Top (Red): +VDC Bottom (Blue): GND"
