File: Solar Panels/Solar Panels.kicad_sch (KiCad schematic)
At the start: 46 parts, among them J1 5040500891

Commit message: August 20th Changes
Finished setting up the PCB board (haven't started the PCB board yet)
Parts:
- D1, D10, D2, D3, D4, D5, D6, D7, D8, D9: footprint (none) -> Solar Panels Library:PMEG10020AELPX
- H1, H2, H3, H4: footprint (none) -> MountingHole:MountingHole_3.2mm_M3_DIN965_Pad
- J1: footprint CON_5040500891 -> Solar Panels Library:CON_5040500891
- JP1, JP2, JP3, JP4: footprint (none) -> Jumper:SolderJumper-2_P1.3mm_Open_Pad1.0x1.5mm
- SC1, SC10, SC11, SC12, SC13, SC14, SC15, SC16, SC17, SC18, SC19, SC2, SC20, SC21, SC22, SC23, SC24, SC25, SC26, SC27, SC3, SC4, SC5, SC6, SC7, SC8, SC9: footprint (none) -> Solar Panels Library:Trisolx Wings
Changed lines of the file:
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@@
 			)
 		)
-		(property "Footprint" ""
+		(property "Footprint" "Solar Panels Library:Trisolx Wings"
 			(at 175.26 65.786 90)
 			(effects
@@
 			)
 		)
-		(property "Footprint" ""
+		(property "Footprint" "Jumper:SolderJumper-2_P1.3mm_Open_Pad1.0x1.5mm"
 			(at 60.96 137.16 0)
 			(effects
@@
 			)
 		)
-		(property "Footprint" ""
+		(property "Footprint" "Solar Panels Library:Trisolx Wings"
 			(at 93.98 65.786 90)
 			(effects
@@
 			)
 		)
-		(property "Footprint" ""
+		(property "Footprint" "Solar Panels Library:PMEG10020AELPX"
 			(at 114.3 44.45 0)
 			(effects
@@
 			)
 		)
-		(property "Footprint" ""
+		(property "Footprint" "Solar Panels Library:Trisolx Wings"
 			(at 72.39 78.486 90)
 			(effects
@@
 			)
 		)
-		(property "Footprint" ""
+		(property "Footprint" "Solar Panels Library:Trisolx Wings"
 			(at 135.89 65.786 90)
 			(effects
@@
 			)
 		)
-		(property "Footprint" ""
+		(property "Footprint" "Solar Panels Library:Trisolx Wings"
 			(at 72.39 65.786 90)
 			(effects
@@
 			)
 		)
-		(property "Footprint" ""
+		(property "Footprint" "MountingHole:MountingHole_3.2mm_M3_DIN965_Pad"
 			(at 29.21 158.75 0)
 			(effects
@@
 			)
 		)
-		(property "Footprint" ""
+		(property "Footprint" "Jumper:SolderJumper-2_P1.3mm_Open_Pad1.0x1.5mm"
 			(at 60.96 170.18 0)
 			(effects
@@
 			)
 		)
-		(property "Footprint" ""
+		(property "Footprint" "Solar Panels Library:Trisolx Wings"
 			(at 175.26 54.356 90)
 			(effects
@@
 			)
 		)
-		(property "Footprint" ""
+		(property "Footprint" "Solar Panels Library:Trisolx Wings"
 			(at 135.89 54.356 90)
 			(effects
@@
 			)
 		)
-		(property "Footprint" ""
+		(property "Footprint" "Solar Panels Library:Trisolx Wings"
 			(at 156.21 78.486 90)
 			(effects
@@
 			)
 		)
-		(property "Footprint" ""
+		(property "Footprint" "Jumper:SolderJumper-2_P1.3mm_Open_Pad1.0x1.5mm"
 			(at 29.21 137.16 0)
 			(effects
@@
 			)
 		)
-		(property "Footprint" ""
+		(property "Footprint" "Solar Panels Library:Trisolx Wings"
 			(at 114.3 78.486 90)
 			(effects
@@
 			)
 		)
-		(property "Footprint" ""
+		(property "Footprint" "Solar Panels Library:Trisolx Wings"
 			(at 52.07 78.486 90)
 			(effects
@@
 			)
 		)
-		(property "Footprint" ""
+		(property "Footprint" "Solar Panels Library:Trisolx Wings"
 			(at 156.21 54.356 90)
 			(effects
@@
 			)
 		)
-		(property "Footprint" ""
+		(property "Footprint" "Solar Panels Library:PMEG10020AELPX"
 			(at 194.31 44.45 0)
 			(effects
@@
 			)
 		)
-		(property "Footprint" ""
+		(property "Footprint" "Solar Panels Library:PMEG10020AELPX"
 			(at 52.07 44.45 0)
 			(effects
@@
 			)
 		)
-		(property "Footprint" ""
+		(property "Footprint" "Solar Panels Library:PMEG10020AELPX"
 			(at 93.98 44.45 0)
 			(effects
@@
 			)
 		)
-		(property "Footprint" ""
+		(property "Footprint" "Solar Panels Library:Trisolx Wings"
 			(at 93.98 54.356 90)
 			(effects
@@
 			)
 		)
-		(property "Footprint" ""
+		(property "Footprint" "Solar Panels Library:PMEG10020AELPX"
 			(at 215.9 58.42 0)
 			(effects
@@
 			)
 		)
-		(property "Footprint" ""
+		(property "Footprint" "Solar Panels Library:Trisolx Wings"
 			(at 93.98 78.486 90)
 			(effects
@@
 			)
 		)
-		(property "Footprint" ""
+		(property "Footprint" "Solar Panels Library:Trisolx Wings"
 			(at 52.07 65.786 90)
 			(effects
@@
 			)
 		)
-		(property "Footprint" ""
+		(property "Footprint" "Solar Panels Library:Trisolx Wings"
 			(at 114.3 54.356 90)
 			(effects
@@
 			)
 		)
-		(property "Footprint" ""
+		(property "Footprint" "MountingHole:MountingHole_3.2mm_M3_DIN965_Pad"
 			(at 60.96 125.73 0)
 			(effects
@@
 			)
 		)
-		(property "Footprint" ""
+		(property "Footprint" "Solar Panels Library:Trisolx Wings"
 			(at 194.31 65.786 90)
 			(effects
@@
 			)
 		)
-		(property "Footprint" ""
+		(property "Footprint" "Solar Panels Library:PMEG10020AELPX"
 			(at 175.26 44.45 0)
 			(effects
@@
 			)
 		)
-		(property "Footprint" "CON_5040500891"
+		(property "Footprint" "Solar Panels Library:CON_5040500891"
 			(at 148.59 132.08 0)
 			(effects
@@
 			)
 		)
-		(property "Footprint" ""
+		(property "Footprint" "Solar Panels Library:Trisolx Wings"
 			(at 194.31 54.356 90)
 			(effects
@@
 			)
 		)
-		(property "Footprint" ""
+		(property "Footprint" "Solar Panels Library:Trisolx Wings"
 			(at 194.31 78.486 90)
 			(effects
@@
 			)
 		)
-		(property "Footprint" ""
+		(property "Footprint" "Solar Panels Library:PMEG10020AELPX"
 			(at 156.21 44.45 0)
 			(effects
@@
 			)
 		)
-		(property "Footprint" ""
+		(property "Footprint" "Solar Panels Library:Trisolx Wings"
 			(at 114.3 65.786 90)
 			(effects
@@
 			)
 		)
-		(property "Footprint" ""
+		(property "Footprint" "Solar Panels Library:PMEG10020AELPX"
 			(at 33.02 44.45 0)
 			(effects
@@
 			)
 		)
-		(property "Footprint" ""
+		(property "Footprint" "Solar Panels Library:Trisolx Wings"
 			(at 33.02 54.356 90)
 			(effects
@@
 			)
 		)
-		(property "Footprint" ""
+		(property "Footprint" "Solar Panels Library:PMEG10020AELPX"
 			(at 72.39 44.45 0)
 			(effects
@@
 			)
 		)
-		(property "Footprint" ""
+		(property "Footprint" "MountingHole:MountingHole_3.2mm_M3_DIN965_Pad"
 			(at 60.96 158.75 0)
 			(effects
@@
 			)
 		)
-		(property "Footprint" ""
+		(property "Footprint" "Solar Panels Library:Trisolx Wings"
 			(at 175.26 78.486 90)
 			(effects
@@
 			)
 		)
-		(property "Footprint" ""
+		(property "Footprint" "Solar Panels Library:Trisolx Wings"
 			(at 52.07 54.356 90)
 			(effects
@@
 			)
 		)
-		(property "Footprint" ""
+		(property "Footprint" "Solar Panels Library:Trisolx Wings"
 			(at 135.89 78.486 90)
 			(effects
@@
 			)
 		)
-		(property "Footprint" ""
+		(property "Footprint" "Solar Panels Library:Trisolx Wings"
 			(at 33.02 78.486 90)
 			(effects
@@
 			)
 		)
-		(property "Footprint" ""
+		(property "Footprint" "Jumper:SolderJumper-2_P1.3mm_Open_Pad1.0x1.5mm"
 			(at 29.21 170.18 0)
 			(effects
@@
 			)
 		)
-		(property "Footprint" ""
+		(property "Footprint" "Solar Panels Library:Trisolx Wings"
 			(at 156.21 65.786 90)
 			(effects
@@
 			)
 		)
-		(property "Footprint" ""
+		(property "Footprint" "Solar Panels Library:Trisolx Wings"
 			(at 33.02 65.786 90)
 			(effects
@@
 			)
 		)
-		(property "Footprint" ""
+		(property "Footprint" "Solar Panels Library:PMEG10020AELPX"
 			(at 135.89 44.45 0)
 			(effects
@@
 			)
 		)
-		(property "Footprint" ""
+		(property "Footprint" "MountingHole:MountingHole_3.2mm_M3_DIN965_Pad"
 			(at 29.21 125.73 0)
 			(effects
@@
 			)
 		)
-		(property "Footprint" ""
+		(property "Footprint" "Solar Panels Library:Trisolx Wings"
 			(at 72.39 54.356 90)
 			(effects
