File: Solar_Panels_1p0U/Solar_Panels_1p0U.kicad_sch (KiCad schematic)
At the start: 46 parts, among them J1 5040500891

Commit message: Kicad 9.0 PCB UPDATE
Parts:
- removed D9: D, Solar Panels Library:PMEG10020AELPX, symbol Device:D
- removed SC25, SC26, SC27: Solar_Cell, Solar Panels Library:Trisolx Wings, symbol Device:Solar_Cell
- SC1, SC10, SC11, SC12, SC13, SC14, SC15, SC16, SC17, SC18, SC19, SC2, SC20, SC21, SC22, SC23, SC24, SC3, SC4, SC5, SC6, SC7, SC8, SC9: footprint Solar Panels Library:Trisolx Wings -> Solar Panels Library:TrisolX Solar Wings
Other:
- moved on the sheet: D10

Commit message: 1u Updates
Parts:
- renumbered D10 to D9
Changed lines of the file:
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@@
 		(dnp no)
 		(fields_autoplaced yes)
-		(property "Reference" "D10"
+		(property "Reference" "D9"
 			(at 196.85 63.4999 90)
 			(effects
@@
 			(project "Solar Panels"
 				(path "/2d09e942-e62e-4d1d-b7bd-24169f5bea3a"
-					(reference "D10")
+					(reference "D9")
 					(unit 1)
 				)
