File: Solar_Panels_1p0U/Solar_Panels_1p0U.kicad_sch (KiCad schematic)
At the start: 46 parts, among them J1 5040500891

Commit message: 1.0U: Layout cells
Parts:
- removed D1, D10, D2, D3, D4, D5, D6, D7, D8, D9: D, Solar Panels Library:PMEG10020AELPX, symbol Device:D
- removed J1: 5040500891, Solar Panels Library:CON_5040500891, symbol Solar Panel:5040500891
- added D11, D2, D4, D6, D8, D9: PMEG3010EP, Solar Panel Library:PMEG10020AELPX, symbol Lib:S3B_R1_00001
- added J1, J3: Conn_01x08_MountingPin, Connector_Molex:Molex_PicoBlade_53261-0871_1x08-1MP_P1.25mm_Horizontal, symbol Connector_Generic_MountingPin:Conn_01x08_MountingPin
- added J4: Conn_01x02, Connector_PinHeader_2.54mm:PinHeader_2x01_P2.54mm_Vertical, symbol Connector_Generic:Conn_01x02
- added J5: Conn_01x08_MountingPin, Connector_Molex:Molex_Pico-Lock_504050-0891_1x08-1MP_P1.50mm_Horizontal, symbol Connector_Generic_MountingPin:Conn_01x08_MountingPin
- added SC28, SC29, SC30: KXOB25-05X3F, Solar Panel Library:KXOB25-05X3F, symbol Device:Solar_Cell
- SC1, SC10, SC11, SC12, SC13, SC14, SC15, SC16, SC17, SC18, SC19, SC2, SC20, SC21, SC22, SC23, SC24, SC25, SC26, SC27, SC3, SC4, SC5, SC6, SC7, SC8, SC9: value Solar_Cell -> KXOB25-05X3F; footprint Solar Panels Library:Trisolx Wings -> Solar Panel Library:KXOB25-05X3F
Connections:
- net +VDC: now also D11.1, D2.1, D4.1, D6.1, D8.1, D9.1, J1.1 (Pin_1), J1.2 (Pin_2), J1.5 (Pin_5), J1.6 (Pin_6), J3.1 (Pin_1), J3.2 (Pin_2), J3.5 (Pin_5), J3.6 (Pin_6), J4.1 (Pin_1), J5.1 (Pin_1), J5.2 (Pin_2), J5.5 (Pin_5), J5.6 (Pin_6)
- net GND: now also D11.2, J1.3 (Pin_3), J1.4 (Pin_4), J1.7 (Pin_7), J1.8 (Pin_8), J1.MP (MountPin), J3.3 (Pin_3), J3.4 (Pin_4), J3.7 (Pin_7), J3.8 (Pin_8), J3.MP (MountPin), J4.2 (Pin_2), J5.3 (Pin_3), J5.4 (Pin_4), J5.7 (Pin_7), J5.8 (Pin_8), J5.MP (MountPin), SC29.2 (-); no longer SC12.2 (-), SC18.2 (-), SC24.2 (-), SC27.2 (-), SC6.2 (-)
- net at SC13.1 (+): now also SC18.2 (-)
- net at SC22.1 (+): now also D8.2
- net at SC16.1 (+): now also D6.2
- net at SC19.1 (+): now also SC24.2 (-)
- net at SC25.1 (+): now also SC30.2 (-)
- net at SC4.1 (+): now also D2.2
- net at SC10.1 (+): now also D4.2
- net at SC1.1 (+): now also SC6.2 (-)
- net at SC7.1 (+): now also SC12.2 (-)
- new net: D9.2, SC30.1 (+)
- new net: SC27.2 (-), SC28.1 (+)
- new net: SC28.2 (-), SC29.1 (+)
Other:
- note added: "Bypass Diode"
- note added: "Power Connector"
- note added: "Solar Cells (6S5P)"
- note removed: "Power"
- note removed: "Solar Panels"
- company: CalgarytoSpace -> CalgaryToSpace
- title: 1U Solar Panels -> 1.25U Solar Panel

Commit message: 1.0U: Finalize layout mostly
Parts:
- removed D9: PMEG3010EP, Solar Panel Library:PMEG10020AELPX, symbol Lib:S3B_R1_00001
- removed J3: Conn_01x08_MountingPin, Connector_Molex:Molex_PicoBlade_53261-0871_1x08-1MP_P1.25mm_Horizontal, symbol Connector_Generic_MountingPin:Conn_01x08_MountingPin
- removed J4: Conn_01x02, Connector_PinHeader_2.54mm:PinHeader_2x01_P2.54mm_Vertical, symbol Connector_Generic:Conn_01x02
- removed SC25, SC26, SC27, SC28, SC29, SC30: KXOB25-05X3F, Solar Panel Library:KXOB25-05X3F, symbol Device:Solar_Cell
- added D1: LED, LED_SMD:LED_0603_1608Metric_Pad1.05x0.95mm_HandSolder, symbol Device:LED
- added J2: PicoBlade_Vertical, Connector_Molex:Molex_PicoBlade_53047-0210_1x02_P1.25mm_Vertical, symbol Connector_Generic:Conn_01x02
- added J6: PicoBlade, Connector_Molex:Molex_PicoBlade_53261-0471_1x04-1MP_P1.25mm_Horizontal, symbol Connector_Generic_MountingPin:Conn_01x04_MountingPin
- added R1: 5k1, Resistor_SMD:R_0603_1608Metric_Pad0.98x0.95mm_HandSolder, symbol Device:R
Connections:
- net GND: now also J6.MP (MountPin)
- new net: J2.1 (Pin_1), J6.1 (Pin_1)
- new net: J2.2 (Pin_2), J6.2 (Pin_2)
- new net: J6.3 (Pin_3), R1.1
- new net: D1.1 (K), J6.4 (Pin_4)
- new net: D1.2 (A), R1.2
Other:
- note added: "Indicator LED and RBF"
- note added: "Solar Cells (6S4P)"
- note removed: "Solar Cells (6S5P)"

Commit message: Finish Rev 3 - 1.0U
Parts:
- renumbered D1 to LED1
Changed lines of the file:
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@@
 		(dnp no)
 		(fields_autoplaced yes)
-		(property "Reference" "D1"
+		(property "Reference" "LED1"
 			(at 232.41 91.7574 90)
 			(effects
@@
 			(project ""
 				(path "/a9ef5d2b-7ce1-4231-ba73-009f8d0b2537"
-					(reference "D1")
+					(reference "LED1")
 					(unit 1)
 				)

Commit message: Finalize Rev 3 of both panels
Other:
- title: 1.25U Solar Panel -> 1.0U Solar Panel
Changed lines of the file:
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@@
 	(paper "USLetter")
 	(title_block
-		(title "1.25U Solar Panel")
-		(date "2025-04-21")
-		(rev "2")
+		(title "1.0U Solar Panel")
+		(date "2025-05-09")
+		(rev "3")
 		(company "CalgaryToSpace")
 	)
