File: Solar_Panels_1p25U/Solar_Panels_1p25U.kicad_pcb (KiCad board)
At the start: 2 copper layers, 113 x 82.5 mm, 56 parts, among them J1 Conn_01x08_MountingPin, J3 Conn_01x08_MountingPin, J4 Conn_01x02, J5 Conn_01x08_MountingPin

Commit message: 1.25U: Fix typo on connector label
Other:
- board text added: "pBlade|pLock"
- board text removed: "pBlade|uLock"
Changed lines of the file:
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@@
 		)
 	)
-	(gr_text "pBlade|uLock"
+	(gr_text "pBlade|pLock"
 		(at 186.5 105 0)
 		(layer "B.SilkS")

Commit message: Finalize Rev 3 of both panels
Parts:
- D11, D2, D4, D6, D8, D9: value PMEG10020AELPX -> PMEG3010EP
Changed lines of the file:
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@@
 	(title_block
 		(title "1.25U Solar Panel")
-		(date "2025-04-21")
-		(rev "2")
+		(date "2025-05-09")
+		(rev "Rev 3")
 		(company "CalgaryToSpace")
 	)
@@
 			)
 		)
-		(property "Description" ""
+		(property "Description" "Single solar cell"
 			(at 0 0 0)
 			(unlocked yes)
@@
 			)
 		)
-		(property "Description" ""
+		(property "Description" "Single solar cell"
 			(at 0 0 0)
 			(unlocked yes)
@@
 			)
 		)
-		(property "Value" "PMEG10020AELPX"
+		(property "Value" "PMEG3010EP"
 			(at 0 1 270)
 			(unlocked yes)
@@
 			)
 		)
-		(property "Description" ""
+		(property "Description" "Single solar cell"
 			(at 0 0 0)
 			(unlocked yes)
@@
 			)
 		)
-		(property "Description" ""
+		(property "Description" "Single solar cell"
 			(at 0 0 0)
 			(unlocked yes)
@@
 			)
 		)
-		(property "Description" ""
+		(property "Description" "Single solar cell"
 			(at 0 0 90)
 			(unlocked yes)
@@
 			)
 		)
-		(property "Description" ""
+		(property "Description" "Single solar cell"
 			(at 0 0 180)
 			(unlocked yes)
@@
 			)
 		)
-		(property "Description" ""
+		(property "Description" "Single solar cell"
 			(at 0 0 0)
 			(unlocked yes)
@@
 			)
 		)
-		(property "Description" ""
+		(property "Description" "Single solar cell"
 			(at 0 0 180)
 			(unlocked yes)
@@
 			)
 		)
-		(property "Description" ""
+		(property "Description" "Single solar cell"
 			(at 0 0 180)
 			(unlocked yes)
@@
 			)
 		)
-		(property "Description" ""
+		(property "Description" "Single solar cell"
 			(at 0 0 180)
 			(unlocked yes)
@@
 			)
 		)
-		(property "Description" ""
+		(property "Description" "Single solar cell"
 			(at 0 0 180)
 			(unlocked yes)
@@
 			)
 		)
-		(property "Value" "PMEG10020AELPX"
+		(property "Value" "PMEG3010EP"
 			(at 0 1 90)
 			(unlocked yes)
@@
 			)
 		)
-		(property "Value" "PMEG10020AELPX"
+		(property "Value" "PMEG3010EP"
 			(at 0 1 180)
 			(unlocked yes)
@@
 			)
 		)
-		(property "Description" ""
+		(property "Description" "Single solar cell"
 			(at 0 0 180)
 			(unlocked yes)
@@
 			)
 		)
-		(property "Description" ""
+		(property "Description" "Single solar cell"
 			(at 0 0 180)
 			(unlocked yes)
@@
 			)
 		)
-		(property "Description" ""
+		(property "Description" "Single solar cell"
 			(at 0 0 90)
 			(unlocked yes)
@@
 			)
 		)
-		(property "Description" ""
+		(property "Description" "Single solar cell"
 			(at 0 0 0)
 			(unlocked yes)
@@
 			)
 		)
-		(property "Description" ""
+		(property "Description" "Single solar cell"
 			(at 0 0 0)
 			(unlocked yes)
@@
 			)
 		)
-		(property "Description" ""
+		(property "Description" "Single solar cell"
 			(at 0 0 0)
 			(unlocked yes)
@@
 			)
 		)
-		(property "Description" ""
+		(property "Description" "Single solar cell"
 			(at 0 0 180)
 			(unlocked yes)
@@
 			)
 		)
-		(property "Description" ""
+		(property "Description" "Single solar cell"
 			(at 0 0 180)
 			(unlocked yes)
@@
 			)
 		)
-		(property "Description" ""
+		(property "Description" "Single solar cell"
 			(at 0 0 0)
 			(unlocked yes)
@@
 			)
 		)
-		(property "Description" ""
+		(property "Description" "Single solar cell"
 			(at 0 0 270)
 			(unlocked yes)
@@
 			)
 		)
-		(property "Description" ""
+		(property "Description" "Single solar cell"
 			(at 0 0 0)
 			(unlocked yes)
@@
 			)
 		)
-		(property "Description" ""
+		(property "Description" "Single solar cell"
 			(at 0 0 180)
 			(unlocked yes)
@@
 			)
 		)
-		(property "Value" "PMEG10020AELPX"
+		(property "Value" "PMEG3010EP"
 			(at 0 1 180)
 			(unlocked yes)
@@
 			)
 		)
-		(property "Description" ""
+		(property "Description" "Single solar cell"
 			(at 0 0 180)
 			(unlocked yes)
@@
 			)
 		)
-		(property "Description" ""
+		(property "Description" "Single solar cell"
 			(at 0 0 180)
 			(unlocked yes)
@@
 			)
 		)
-		(property "Description" ""
+		(property "Description" "Single solar cell"
 			(at 0 0 0)
 			(unlocked yes)
@@
 			)
 		)
-		(property "Value" "PMEG10020AELPX"
+		(property "Value" "PMEG3010EP"
 			(at 0 1 180)
 			(unlocked yes)
@@
 			)
 		)
-		(property "Description" ""
+		(property "Description" "Single solar cell"
 			(at 0 0 180)
 			(unlocked yes)
@@
 			)
 		)
-		(property "Description" ""
+		(property "Description" "Single solar cell"
 			(at 0 0 0)
 			(unlocked yes)
@@
 			)
 		)
-		(property "Description" ""
+		(property "Description" "Single solar cell"
 			(at 0 0 180)
 			(unlocked yes)
@@
 			)
 		)
-		(property "Description" ""
+		(property "Description" "Single solar cell"
 			(at 0 0 180)
 			(unlocked yes)
@@
 			)
 		)
-		(property "Value" "PMEG10020AELPX"
+		(property "Value" "PMEG3010EP"
 			(at 0 1 180)
 			(unlocked yes)
